File: power.kicad_sch (KiCad schematic)
At the start: 22 parts, among them U3 AP62250Z6

Commit message: Bom updates
Parts:
- C10: MPN (none) -> CL05B104KP5NNNC; Package (none) -> 0402
- C11, C12: MPN (none) -> CL21A226MAYNNNE; Package (none) -> 0805
- C17, C18: MPN (none) -> CC0603KRX7R7BB104; Package (none) -> 0603
- C9: MPN (none) -> CL21A106KOQNNNE; Package (none) -> 0805
- D10, D4: MPN (none) -> LTST-C190KFKT; Package (none) -> 0603
- D8: MPN (none) -> S1J-13-F; Package (none) -> SMA
- FL1: MPN (none) -> 0603USB-222MLC
- L1: MPN (none) -> SRP5030TA-2R2M
- R10: MPN (none) -> RT0402FRE0731K6L; Package (none) -> 0402
- R11, R9: MPN (none) -> RC0402JR-0710KL; Package (none) -> 0402
- R12: MPN (none) -> ERJ-6DSFR10V; Package (none) -> 0805
- R16, R50: MPN (none) -> RC0402FR-070RL; Package (none) -> 0402
- R28: MPN (none) -> RC0402JR-071KL; Package (none) -> 0402
- R54: Package (none) -> 0402
- TP17, TP20: now not fitted
- U3: MPN (none) -> AP62250Z6-7; Package (none) -> SOT-563

Commit message: Launch day
Completed BOM, added silk art
Parts:
- R54: MPN (none) -> ERA-2AEB302X
Changed lines of the file:
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@@
+			)
+		)
+		(property "MPN" "ERA-2AEB302X"
+			(at 27.94 73.66 0)
+			(effects
+				(font
+					(size 1.27 1.27)
+				)
+				(hide yes)
 			)
 		)
