File: raspi.kicad_sch (KiCad schematic)
At the start: 54 parts, among them J8 Conn_01x03, J9 debug_probe, Q2 Q_NPN_BCE, SW1 SW_Omron_B3FS, U6 RP2350B-QFN80, U8 IS25LP040E-JNLE-TR, U9 IS25LP040E-JNLE-TR, X1 ASE-12.000MHZ-L-C-T

Commit message: Launch day
Completed BOM, added silk art
Parts:
- R47, R56: MPN (none) -> RC0402FR-0710RL
- R48, R49: MPN (none) -> RC0402FR-07100RL
Changed lines of the file:
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@@
 			)
 		)
+		(property "MPN" "RC0402FR-07100RL"
+			(at 30.48 148.59 0)
+			(effects
+				(font
+					(size 1.27 1.27)
+				)
+				(hide yes)
+			)
+		)
 		(pin "2"
 		)
@@
 			)
 		)
+		(property "MPN" "RC0402FR-07100RL"
+			(at 30.48 143.51 0)
+			(effects
+				(font
+					(size 1.27 1.27)
+				)
+				(hide yes)
+			)
+		)
 		(pin "2"
 		)
@@
 			)
 		)
+		(property "MPN" "RC0402FR-0710RL"
+			(at 264.16 64.77 0)
+			(effects
+				(font
+					(size 1.27 1.27)
+				)
+				(hide yes)
+			)
+		)
 		(pin "1"
 		)
@@
 			(at 139.7 21.59 0)
 			(effects
+				(font
+					(size 1.27 1.27)
+				)
+				(hide yes)
+			)
+		)
+		(property "MPN" "RC0402FR-0710RL"
+			(at 139.7 21.59 0)
+			(effects
